File: PCBs/Control/Control.sch (KiCad schematic (older format))
At the start: 33 parts, among them J1 Conn_01x06, SW1 SW_Push, SW2 SW_Push, SW3 SW_Push, SW4 SW_Push, SW5 SW_Push, SW6 SW_Push, U1 ISO7341C

Commit message: Add sd card
Parts:
- B1: symbol Arduino_Module_Custom:Micro_SD_Card_Module -> Control-rescue:Micro_SD_Card_Module-Arduino_Module_Custom
- B2: symbol MCU_Module_Custom:DOIT_ESP32_Devkit_v1 -> Control-rescue:DOIT_ESP32_Devkit_v1-MCU_Module_Custom
- B?: symbol SparkFun-Boards:ARDUINO_PRO_MINI -> Control-rescue:ARDUINO_PRO_MINI-SparkFun-Boards
- DS1: symbol Arduino_Module_Custom:128x64_OLED_Display -> Control-rescue:128x64_OLED_Display-Arduino_Module_Custom
- PS1: symbol RFM-0505S:RFM-0505S -> Control-rescue:RFM-0505S-RFM-0505S
Changed lines of the file:
@@
 	1300 1700 1200 1700
 $Comp
-L MCU_Module_Custom:DOIT_ESP32_Devkit_v1 B2
+L Control-rescue:DOIT_ESP32_Devkit_v1-MCU_Module_Custom B2
 U 1 1 5BF7BA5F
 P 4950 1300
@@
 	1700 3650 1550 3650
 $Comp
-L RFM-0505S:RFM-0505S PS1
+L Control-rescue:RFM-0505S-RFM-0505S PS1
 U 1 1 5BF39FF2
 P 1900 1300
@@
 $EndComp
 $Comp
-L Arduino_Module_Custom:128x64_OLED_Display DS1
+L Control-rescue:128x64_OLED_Display-Arduino_Module_Custom DS1
 U 1 1 5BF42832
 P 10000 1400
@@
 	5800 2500 5950 2500
 $Comp
-L Arduino_Module_Custom:Micro_SD_Card_Module B1
+L Control-rescue:Micro_SD_Card_Module-Arduino_Module_Custom B1
 U 1 1 5BF75232
 P 1850 5000
@@
 	10150 1850 10150 2250
 $Comp
-L SparkFun-Boards:ARDUINO_PRO_MINI B?
+L Control-rescue:ARDUINO_PRO_MINI-SparkFun-Boards B?
 U 1 1 5C01C3E7
 P 8450 1800
