File: PCBs/Infrared/Infrared.kicad_pcb (KiCad board)
At the start: 2 copper layers, 207 x 91.1 mm, 20 parts, among them J1 Conn_01x05_Male, Q1 Q_PNP_CBE, U1 LD1117S33TR_SOT223, U2 ESP-32S

Commit message: Infared PCB
Parts:
- removed REF** (x4): MountingHole_3.2mm_M3_DIN965, MountingHole:MountingHole_3.2mm_M3_DIN965
- added H1: MountingHole, MountingHole:MountingHole_3.2mm_M3_DIN965, F.Cu at (15.0, 15.0)
- added H2: MountingHole, MountingHole:MountingHole_3.2mm_M3_DIN965, F.Cu at (79.0, 79.0)
- added H3: MountingHole, MountingHole:MountingHole_3.2mm_M3_DIN965, F.Cu at (15.0, 79.0)
- added H4: MountingHole, MountingHole:MountingHole_3.2mm_M3_DIN965, F.Cu at (79.0, 15.0)
- added U3: SHT3X_Breakout_Board, Connector_PinHeader_2.54mm:PinHeader_1x04_P2.54mm_Vertical, F.Cu at (15.0, 51.6)
- moved C2 34.8 mm to (64.0, 34.6)
- moved D1 34.8 mm to (63.0, 44.0)
- moved D2 34.8 mm to (71.6, 42.0)
- moved D3 34.8 mm to (77.5, 49.7)
- moved D4 34.8 mm to (67.6, 49.1)
- moved D5 34.8 mm to (59.6, 47.8)
- moved D6 34.8 mm to (72.0, 55.5)
- moved J1 34.8 mm to (76.9, 33.7)
- moved Q1 34.8 mm to (57.9, 66.0)
- moved R1 34.8 mm to (63.4, 64.1)
- moved R2 34.8 mm to (29.2, 55.9)
- moved R3 34.8 mm to (63.4, 67.1)
- moved U1 34.8 mm to (58.8, 37.1)
- moved U2 34.8 mm to (35.6, 47.5)
- moved C1 34.8 mm to (56.2, 25.6)
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Connections:
- U2 pad 1: Net-(U2-Pad1) -> +3V3
- U2 pad 11: Net-(U2-Pad11) -> SDA
- U2 pad 14: Net-(U2-Pad14) -> SCL
Routing:
- net SDA: track 0.00 -> 45.1 mm
- net +3V3: track 0.00 -> 21.4 mm
- net SCL: track 0.00 -> 19.8 mm
Other:
- board size 207 x 91.1 mm -> 70 x 70 mm

Commit message: layer 2 update
Parts:
- J1: footprint Connector_PinHeader_2.54mm:PinHeader_1x05_P2.54mm_Vertical -> MIcro_USB:PinHeader_1x05_P2.54mm_Vertical
- moved J1 22.5 mm to (64.3, 15.0), turned to 90 degrees
- moved H2 16.7 mm to (67.2, 67.2)
- moved C1 16.7 mm to (44.4, 13.8)
- moved D2 16.7 mm to (59.9, 30.2)
- moved D4 16.7 mm to (55.8, 37.3)
- moved D7 16.7 mm to (51.7, 42.2)
- moved H1 16.7 mm to (3.22, 3.22)
- moved H3 16.7 mm to (3.22, 67.2)
- moved H4 16.7 mm to (67.2, 3.22)
- moved Q1 16.7 mm to (46.2, 54.2)
- moved R3 16.7 mm to (51.6, 55.3)
- moved U1 16.7 mm to (47.0, 25.4)
- moved D1 16.7 mm to (51.2, 32.2)
- moved D3 16.7 mm to (65.7, 37.9)
- moved D5 16.7 mm to (47.8, 36.0)
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Routing:
- net +5V: track 38.9 -> 33.7 mm
- net Net-(C2-Pad1): track 37.9 -> 42.9 mm
