File: PCBs/Layer1/Layer1.sch (KiCad schematic (older format))
At the start: 46 parts, among them J1 Screw_Terminal_01x02, J2 Conn_01x12, T1 T60404-E4624-X501, U1 STPM_STPM10BTR, U2 level_shifter, U3 Micro_SD_Shield, U4 DOIT_ESP32_Devkit_v1-MCU_Modu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, Y1 4.194304 MHz

Commit message: Layer1 Ver1.0
Connections:
- net MOSI: no longer U3.16 (TX)
- no-connect marks 30 -> 31
Changed lines of the file:
@@
 Text Label 5350 6800 2    50   ~ 0
 MOSI
-Text GLabel 2150 5900 0    50   Input ~ 0
-MOSI
-Wire Wire Line
-	2150 5900 2300 5900
+NoConn ~ 2300 5900
 $EndSCHEMATC

Commit message: WIP: version 2
Parts:
- removed PS1: RAC05-05SK, RAC05-05SK:RAC05-12SK, symbol RAC05-05SK:RAC05-05SK
- added C?: 1nF, symbol Device:C
- added C?: 470nF 630V, symbol Device:C
- added C?: 4700uF, symbol Device:CP
- added D2, D3, D4: LED_Small, LED_SMD:LED_0603_1608Metric_Pad1.05x0.95mm_HandSolder, symbol Device:LED_Small
- added D? (x2): 600V 1A, symbol Device:D
- added D?: 5.1V, symbol Device:D_Zener
- added J?: Screw_Terminal_01x02, TerminalBlock:TerminalBlock_bornier-2_P5.08mm, symbol Connector:Screw_Terminal_01x02
- added L?: 220uH, symbol Device:L
- added L?: 1uH, symbol Device:L
- added PS?: RAC05-05SK, RAC05-12SK, symbol RAC05-05SK:RAC05-05SK
- added R20, R21, R22: 6.8K, Resistor_SMD:R_0603_1608Metric_Pad1.05x0.95mm_HandSolder, symbol Device:R_Small
- added R?: 82R 2W, symbol Device:R
- added R?: 0R, symbol Device:R
- C3, C4, C5, C6: footprint Capacitor_SMD:C_1206_3216Metric_Pad1.42x1.75mm_HandSolder -> Capacitor_SMD:C_0603_1608Metric_Pad1.05x0.95mm_HandSolder
Connections:
- net V_IN is gone; now on net GND: C7.2, J1.2 (Pin_2), R5.2, R8.2, RV1.2, TP2.1, U1.14 (V_IN)
- net +5V: now also C?.1, D2.2 (A), D3.2 (A), D4.2 (A), D?.1 (K), D?.1 (K); no longer U4.15 (VIN)
- net GND: now also U1.11 (I_IP2), U1.12 (I_IN2), C?.2, C?.2, D?.2 (A), D?.2 (A), L?.1, L?.2; no longer U2.3 (GND), U3.10 (GND), U4.14 (GND)
- net L: now also L?.1
- net STPM10_SCL: now also R21.1
- net STPM10_SDA: now also R22.1
- net STPM10_SYN: now also R20.1
- net V_IP: now also R?.1; no longer R4.1, R5.1, R7.1
- new net: R4.1, R5.1, R7.1, R?.2
- new net: D2.1 (K), R20.2
- new net: C?.1, L?.2, R?.2
- new net: C?.2, R?.1
- new net: C?.1, D?.1 (K), D?.2 (A)
- new net: D3.1 (K), R21.2
- new net: D4.1 (K), R22.2
- new net: J?.1 (Pin_1), PS?.1 (VAC_IN_(L))
- new net: J?.2 (Pin_2), PS?.2 (VAC_IN_(N))
- new net +5VD: PS?.4 (-VOUT), U4.15 (VIN)
- new net GNDD: PS?.5 (+VOUT), U2.3 (GND), U3.10 (GND), U4.14 (GND)
- no-connect marks 31 -> 28
Other:
- moved on the sheet: C7, H1, H2, H3, H4, J2, R16, R17, R18, R19, R5, R6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

Commit message: WIP: version 2 schematics
Parts:
- C10: renamed from C?; footprint (none) -> Capacitor_SMD:C_1806_4516Metric_Pad1.57x1.80mm_HandSolder
- C11: renamed from C?; footprint (none) -> Capacitor_THT:CP_Radial_D12.5mm_P5.00mm
- C9: renamed from C?; footprint (none) -> Layer1:C_Rect_L26.5mm_W15.5mm_P22.50mm_MKS4
- D5, D6: renamed from D?; footprint (none) -> Diode_SMD:D_SMA_Handsoldering
- D7: renamed from D?; footprint (none) -> Layer1:SOD-80
- L1, L2: renamed from L?; footprint (none) -> Inductor_SMD:L_1812_4532Metric_Pad1.30x3.40mm_HandSolder
- PS1: renamed from PS?; footprint RAC05-12SK -> RAC05-05SK:RAC05-12SK
- R23: renamed from R?; footprint (none) -> Resistor_THT:R_Axial_DIN0617_L17.0mm_D6.0mm_P20.32mm_Horizontal
- R24: renamed from R?; footprint (none) -> Resistor_SMD:R_1206_3216Metric_Pad1.42x1.75mm_HandSolder
- gave numbers to parts that had none: 1
Connections:
- net GND: no longer J2.2 (Pin_2)
- net GNDD: now also J2.2 (Pin_2)
Changed lines of the file:
@@
 Wire Wire Line
 	3250 4150 3250 5000
-$Comp
-L power:GND #PWR014
-U 1 1 5C8A4C1B
-P 900 5650
-F 0 "#PWR014" H 900 5400 50  0001 C CNN
-F 1 "GND" H 905 5477 50  0000 C CNN
-F 2 "" H 900 5650 50  0001 C CNN
-F 3 "" H 900 5650 50  0001 C CNN
-	1    900  5650
-	1    0    0    -1
-$EndComp
 Wire Wire Line
 	900  5450 900  5650
-$Comp
-L power:GND #PWR06
-U 1 1 5C8A6E0D
-P 6650 2450
-F 0 "#PWR06" H 6650 2200 50  0001 C CNN
-F 1 "GND" H 6655 2277 50  0000 C CNN
-F 2 "" H 6650 2450 50  0001 C CNN
-F 3 "" H 6650 2450 50  0001 C CNN
-	1    6650 2450
-	1    0    0    -1
-$EndComp
 $Comp
 L power:GND #PWR05
@@
 	9700 2850 9700 3000
 Wire Wire Line
-	9700 3000 10000 3000
-Wire Wire Line
 	10300 3000 10300 2850
-$Comp
-L power:GND #PWR07
-U 1 1 5C8B2200
-P 10000 3000
-F 0 "#PWR07" H 10000 2750 50  0001 C CNN
-F 1 "GND" H 10005 2827 50  0000 C CNN
-F 2 "" H 10000 3000 50  0001 C CNN
-F 3 "" H 10000 3000 50  0001 C CNN
-	1    10000 3000
-	1    0    0    -1
-$EndComp
-Connection ~ 10000 3000
-Wire Wire Line
-	10000 3000 10300 3000
 Wire Wire Line
 	9700 2400 9700 2000
@@
 	1    8850 9150
 	-1   0    0    -1
-$EndComp
-$Comp
-L power:GND #PWR09
-U 1 1 5CB45669
-P 8600 9150
-F 0 "#PWR09" H 8600 8900 50  0001 C CNN
-F 1 "GND" H 8605 8977 50  0000 C CNN
-F 2 "" H 8600 9150 50  0001 C CNN
-F 3 "" H 8600 9150 50  0001 C CNN
-	1    8600 9150
-	1    0    0    1
 $EndComp
 Wire Wire Line
@@
 	8350 1850 8700 1850
 $Comp
-L power:GND #PWR?
+L power:GND #PWR011
 U 1 1 5C91DF01
 P 8450 2400
-F 0 "#PWR?" H 8450 2150 50  0001 C CNN
+F 0 "#PWR011" H 8450 2150 50  0001 C CNN
 F 1 "GND" H 8455 2227 50  0000 C CNN
 F 2 "" H 8450 2400 50  0001 C CNN
@@
 	8450 2250 8450 2400
 $Comp
-L Device:C C?
+L Device:C C10
 U 1 1 5C8C30BE
 P 2250 1700
-F 0 "C?" H 2365 1746 50  0000 L CNN
+F 0 "C10" H 2365 1746 50  0000 L CNN
 F 1 "1nF" H 2365 1655 50  0000 L CNN
-F 2 "" H 2288 1550 50  0001 C CNN
+F 2 "Capacitor_SMD:C_1806_4516Metric_Pad1.57x1.80mm_HandSolder" H 2288 1550 50  0001 C CNN
 F 3 "~" H 2250 1700 50  0001 C CNN
 	1    2250 1700
@@
 $EndComp
 $Comp
-L Device:L L?
+L Device:L L1
 U 1 1 5C8C3301
 P 2000 1550
-F 0 "L?" V 2190 1550 50  0000 C CNN
+F 0 "L1" V 2190 1550 50  0000 C CNN
 F 1 "220uH" V 2099 1550 50  0000 C CNN
-F 2 "" H 2000 1550 50  0001 C CNN
+F 2 "Inductor_SMD:L_1812_4532Metric_Pad1.30x3.40mm_HandSolder" H 2000 1550 50  0001 C CNN
 F 3 "~" H 2000 1550 50  0001 C CNN
 	1    2000 1550
@@
 $EndComp
 $Comp
-L Device:R R?
+L Device:R R23
 U 1 1 5C8C3626
 P 2500 1550
-F 0 "R?" V 2293 1550 50  0000 C CNN
+F 0 "R23" V 2293 1550 50  0000 C CNN
 F 1 "82R 2W" V 2384 1550 50  0000 C CNN
-F 2 "" V 2430 1550 50  0001 C CNN
+F 2 "Resistor_THT:R_Axial_DIN0617_L17.0mm_D6.0mm_P20.32mm_Horizontal" V 2430 1550 50  0001 C CNN
 F 3 "~" H 2500 1550 50  0001 C CNN
 	1    2500 1550
@@
 $EndComp
 $Comp
-L Device:C C?
+L Device:C C9
 U 1 1 5C8C37C8
 P 2900 1550
-F 0 "C?" V 2648 1550 50  0000 C CNN
+F 0 "C9" V 2648 1550 50  0000 C CNN
 F 1 "470nF 630V" V 2739 1550 50  0000 C CNN
-F 2 "" H 2938 1400 50  0001 C CNN
+F 2 "Layer1:C_Rect_L26.5mm_W15.5mm_P22.50mm_MKS4" H 2938 1400 50  0001 C CNN
 F 3 "~" H 2900 1550 50  0001 C CNN
 	1    2900 1550
@@
 $EndComp
 $Comp
-L Device:D D?
+L Device:D D6
 U 1 1 5C8C3C35
 P 3150 1700
-F 0 "D?" V 3104 1779 50  0000 L CNN
+F 0 "D6" V 3104 1779 50  0000 L CNN
 F 1 "600V 1A" V 3195 1779 50  0000 L CNN
-F 2 "" H 3150 1700 50  0001 C CNN
+F 2 "Diode_SMD:D_SMA_Handsoldering" H 3150 1700 50  0001 C CNN
 F 3 "~" H 3150 1700 50  0001 C CNN
 	1    3150 1700
@@
 $EndComp
 $Comp
-L Device:D D?
+L Device:D D5
 U 1 1 5C8C3D88
 P 3400 1550
-F 0 "D?" H 3400 1334 50  0000 C CNN
+F 0 "D5" H 3400 1334 50  0000 C CNN
 F 1 "600V 1A" H 3400 1425 50  0000 C CNN
-F 2 "" H 3400 1550 50  0001 C CNN
+F 2 "Diode_SMD:D_SMA_Handsoldering" H 3400 1550 50  0001 C CNN
 F 3 "~" H 3400 1550 50  0001 C CNN
 	1    3400 1550
@@
 $EndComp
 $Comp
-L Device:CP C?
+L Device:CP C11
 U 1 1 5C8C4107
 P 3650 1700
-F 0 "C?" H 3768 1746 50  0000 L CNN
+F 0 "C11" H 3768 1746 50  0000 L CNN
 F 1 "4700uF" H 3768 1655 50  0000 L CNN
-F 2 "" H 3688 1550 50  0001 C CNN
+F 2 "Capacitor_THT:CP_Radial_D12.5mm_P5.00mm" H 3688 1550 50  0001 C CNN
 F 3 "~" H 3650 1700 50  0001 C CNN
 	1    3650 1700
@@
 $EndComp
 $Comp
-L Device:D_Zener D?
+L Device:D_Zener D7
 U 1 1 5C8E9FF8
 P 4150 1700
-F 0 "D?" V 4104 1779 50  0000 L CNN
+F 0 "D7" V 4104 1779 50  0000 L CNN
 F 1 "5.1V" V 4195 1779 50  0000 L CNN
-F 2 "" H 4150 1700 50  0001 C CNN
+F 2 "Layer1:SOD-80" H 4150 1700 50  0001 C CNN
 F 3 "~" H 4150 1700 50  0001 C CNN
 	1    4150 1700
@@
 Connection ~ 1600 1850
 $Comp
-L power:+5V #PWR?
+L power:+5V #PWR02
 U 1 1 5C96F276
 P 4150 1450
-F 0 "#PWR?" H 4150 1300 50  0001 C CNN
+F 0 "#PWR02" H 4150 1300 50  0001 C CNN
 F 1 "+5V" H 4165 1623 50  0000 C CNN
 F 2 "" H 4150 1450 50  0001 C CNN
@@
 Connection ~ 4150 1550
 $Comp
-L power:GND #PWR?
+L power:GND #PWR03
 U 1 1 5C97A703
 P 4150 1950
-F 0 "#PWR?" H 4150 1700 50  0001 C CNN
+F 0 "#PWR03" H 4150 1700 50  0001 C CNN
 F 1 "GND" H 4155 1777 50  0000 C CNN
 F 2 "" H 4150 1950 50  0001 C CNN
@@
 Connection ~ 4150 1850
 $Comp
-L Device:L L?
+L Device:L L2
 U 1 1 5C985D5E
 P 4500 1850
-F 0 "L?" V 4690 1850 50  0000 C CNN
+F 0 "L2" V 4690 1850 50  0000 C CNN
 F 1 "1uH" V 4599 1850 50  0000 C CNN
-F 2 "" H 4500 1850 50  0001 C CNN
+F 2 "Inductor_SMD:L_1812_4532Metric_Pad1.30x3.40mm_HandSolder" H 4500 1850 50  0001 C CNN
 F 3 "~" H 4500 1850 50  0001 C CNN
 	1    4500 1850
@@
 	4150 1850 4350 1850
 $Comp
-L power:GNDA #PWR?
+L power:GNDA #PWR08
 U 1 1 5C991886
 P 4800 1950
-F 0 "#PWR?" H 4800 1700 50  0001 C CNN
+F 0 "#PWR08" H 4800 1700 50  0001 C CNN
 F 1 "GNDA" H 4805 1777 50  0000 C CNN
 F 2 "" H 4800 1950 50  0001 C CNN
@@
 	4800 1850 4800 1950
 $Comp
-L power:GNDA #PWR?
+L power:GNDA #PWR012
 U 1 1 5C99DACC
 P 2700 3650
-F 0 "#PWR?" H 2700 3400 50  0001 C CNN
+F 0 "#PWR012" H 2700 3400 50  0001 C CNN
 F 1 "GNDA" H 2705 3477 50  0000 C CNN
 F 2 "" H 2700 3650 50  0001 C CNN
@@
 	3350 3500 4150 3500
 $Comp
-L Device:R R?
+L Device:R R24
 U 1 1 5C922934
 P 3750 2500
-F 0 "R?" V 3543 2500 50  0000 C CNN
+F 0 "R24" V 3543 2500 50  0000 C CNN
 F 1 "0R" V 3634 2500 50  0000 C CNN
-F 2 "" V 3680 2500 50  0001 C CNN
+F 2 "Resistor_SMD:R_1206_3216Metric_Pad1.42x1.75mm_HandSolder" V 3680 2500 50  0001 C CNN
 F 3 "~" H 3750 2500 50  0001 C CNN
 	1    3750 2500
@@
 Connection ~ 4150 2500
 $Comp
-L RAC05-05SK:RAC05-05SK PS?
+L RAC05-05SK:RAC05-05SK PS1
 U 1 1 5C93E1F0
 P 1150 8300
-F 0 "PS?" H 1900 8565 50  0000 C CNN
+F 0 "PS1" H 1900 8565 50  0000 C CNN
 F 1 "RAC05-05SK" H 1900 8474 50  0000 C CNN
-F 2 "RAC05-12SK" H 2500 8400 50  0001 L CNN
+F 2 "RAC05-05SK:RAC05-12SK" H 2500 8400 50  0001 L CNN
 F 3 "http://www.mouser.com/datasheet/2/468/RAC05-K-1140238.pdf" H 2500 8300 50  0001 L CNN
 F 4 "Recom 5W Encapsulated Switch Mode Power Supply, 1A, 5V dc" H 2500 8200 50  0001 L CNN "Description"
@@
 	3250 3850 3250 3000
 $Comp
-L Connector:Screw_Terminal_01x02 J?
+L Connector:Screw_Terminal_01x02 J3
 U 1 1 5C99D16D
 P 850 8300
-F 0 "J?" V 816 8380 50  0000 L CNN
+F 0 "J3" V 816 8380 50  0000 L CNN
 F 1 "Screw_Terminal_01x02" V 725 8380 50  0000 L CNN
 F 2 "TerminalBlock:TerminalBlock_bornier-2_P5.08mm" H 850 8300 50  0001 C CNN
@@
 $EndComp
 $Comp
-L power:+5VD #PWR?
+L power:+5VD #PWR015
 U 1 1 5C9CB185
 P 2800 8150
-F 0 "#PWR?" H 2800 8000 50  0001 C CNN
+F 0 "#PWR015" H 2800 8000 50  0001 C CNN
 F 1 "+5VD" H 2815 8323 50  0000 C CNN
 F 2 "" H 2800 8150 50  0001 C CNN
@@
 	2800 8300 2650 8300
 $Comp
-L power:GNDD #PWR?
+L power:GNDD #PWR019
 U 1 1 5C9D92A8
 P 2800 8550
-F 0 "#PWR?" H 2800 8300 50  0001 C CNN
+F 0 "#PWR019" H 2800 8300 50  0001 C CNN
 F 1 "GNDD" H 2804 8395 50  0000 C CNN
 F 2 "" H 2800 8550 50  0001 C CNN
@@
 	2800 8400 2800 8550
 $Comp
-L power:+5VD #PWR?
+L power:+5VD #PWR021
 U 1 1 5C9E757C
 P 5250 8800
-F 0 "#PWR?" H 5250 8650 50  0001 C CNN
+F 0 "#PWR021" H 5250 8650 50  0001 C CNN
 F 1 "+5VD" H 5265 8973 50  0000 C CNN
 F 2 "" H 5250 8800 50  0001 C CNN
@@
 $EndComp
 $Comp
-L power:GNDD #PWR?
+L power:GNDD #PWR022
 U 1 1 5C9E7685
 P 5550 8800
-F 0 "#PWR?" H 5550 8550 50  0001 C CNN
+F 0 "#PWR022" H 5550 8550 50  0001 C CNN
 F 1 "GNDD" H 5554 8645 50  0000 C CNN
 F 2 "" H 5550 8800 50  0001 C CNN
@@
 	5100 9050 5550 9050
 $Comp
-L power:GNDD #PWR?
+L power:GNDD #PWR024
 U 1 1 5C9F5FC8
 P 800 10150
-F 0 "#PWR?" H 800 9900 50  0001 C CNN
+F 0 "#PWR024" H 800 9900 50  0001 C CNN
 F 1 "GNDD" H 804 9995 50  0000 C CNN
 F 2 "" H 800 10150 50  0001 C CNN
@@
 $EndComp
 $Comp
-L power:GNDD #PWR?
+L power:GNDD #PWR023
 U 1 1 5C9F6D2A
 P 6150 9350
-F 0 "#PWR?" H 6150 9100 50  0001 C CNN
+F 0 "#PWR023" H 6150 9100 50  0001 C CNN
 F 1 "GNDD" V 6154 9240 50  0000 R CNN
 F 2 "" H 6150 9350 50  0001 C CNN
@@
 Wire Wire Line
 	1050 8400 1150 8400
+$Comp
+L power:GNDD #PWR?
+U 1 1 5CA6FBEC
+P 8600 9150
+F 0 "#PWR?" H 8600 8900 50  0001 C CNN
+F 1 "GNDD" H 8604 8995 50  0000 C CNN
+F 2 "" H 8600 9150 50  0001 C CNN
+F 3 "" H 8600 9150 50  0001 C CNN
+	1    8600 9150
+	-1   0    0    1
+$EndComp
+$Comp
+L power:GNDA #PWR?
+U 1 1 5CA7119F
+P 6650 2450
+F 0 "#PWR?" H 6650 2200 50  0001 C CNN
+F 1 "GNDA" H 6655 2277 50  0000 C CNN
+F 2 "" H 6650 2450 50  0001 C CNN
+F 3 "" H 6650 2450 50  0001 C CNN
+	1    6650 2450
+	1    0    0    -1
+$EndComp
+$Comp
+L power:GNDA #PWR?
+U 1 1 5CA715AF
+P 10000 3000
+F 0 "#PWR?" H 10000 2750 50  0001 C CNN
+F 1 "GNDA" H 10005 2827 50  0000 C CNN
+F 2 "" H 10000 3000 50  0001 C CNN
+F 3 "" H 10000 3000 50  0001 C CNN
+	1    10000 3000
+	1    0    0    -1
+$EndComp
+Wire Wire Line
+	9700 3000 10000 3000
+Connection ~ 10000 3000
+Wire Wire Line
+	10000 3000 10300 3000
+$Comp
+L power:GNDA #PWR?
+U 1 1 5CA71E10
+P 900 5650
+F 0 "#PWR?" H 900 5400 50  0001 C CNN
+F 1 "GNDA" H 905 5477 50  0000 C CNN
+F 2 "" H 900 5650 50  0001 C CNN
+F 3 "" H 900 5650 50  0001 C CNN
+	1    900  5650
+	1    0    0    -1
+$EndComp
 $EndSCHEMATC

Commit message: Layer 1 Ver2, waiting for  review
Parts:
- added H5, H6: MountingHole, MountingHole:MountingHole_2.7mm_M2.5_DIN965, symbol Mechanical:MountingHole
- added J4, J5: Conn_01x06, Connector_PinHeader_2.54mm:PinHeader_1x06_P2.54mm_Vertical, symbol Connector_Generic:Conn_01x06
- added TP5: TestPoint, TestPoint:TestPoint_THTPad_2.0x2.0mm_Drill1.0mm, symbol Connector:TestPoint
Connections:
- net +5V: now also J4.4 (Pin_4), J5.4 (Pin_4); no longer J2.1 (Pin_1)
- net +5VD: now also J2.1 (Pin_1)
- net ESP32_SCS: now also U2.6 (LV1); no longer U2.5 (LV2)
- net ESP32_SDA: now also U2.1 (LV4); no longer U2.6 (LV1)
- net ESP32_SYN: now also U2.5 (LV2); no longer U2.1 (LV4)
- net GND: now also J4.3 (Pin_3), J5.3 (Pin_3); no longer C1.2, C10.2, C11.2, C2.2, C3.2, C4.2, C5.1, C6.1, C7.2, D6.2 (A), D7.2 (A), J1.2 (Pin_2), L2.1, R14.2, R5.2, R8.2, RV1.2, TP2.1, U1.11 (I_IP2), U1.12 (I_IN2), U1.14 (V_IN), U1.5 (VSS)
- net STPM10_LED: now also TP5.1; no longer J2.12 (Pin_12)
- net STPM10_SCL: now also J4.2 (Pin_2), J5.2 (Pin_2)
- net STPM10_SCS: now also U2.7 (HV1), J4.6 (Pin_6), J5.6 (Pin_6); no longer U2.8 (HV2)
- net STPM10_SDA: now also U2.12 (HV4), J4.1 (Pin_1), J5.1 (Pin_1); no longer U2.7 (HV1)
- net STPM10_SYN: now also U2.8 (HV2), J4.5 (Pin_5), J5.5 (Pin_5); no longer U2.12 (HV4)
- new net GNDREF: C1.2, C10.2, C11.2, C2.2, C3.2, C4.2, C5.1, C6.1, C7.2, D6.2 (A), D7.2 (A), J1.2 (Pin_2), L2.1, R14.2, R5.2, R8.2, RV1.2, TP2.1, U1.14 (V_IN), U1.5 (VSS)
- no-connect marks 28 -> 31

Commit message: WIP add pinheader
Parts:
- added J10, J11, J12, J13, J14, J15, J16, J17, J6, J7, J8, J9: Conn_01x02, Connector_PinHeader_2.54mm:PinHeader_1x02_P2.54mm_Vertical, symbol Connector_Generic:Conn_01x02
Connections:
- net +5V: now also J17.1 (Pin_1), J8.2 (Pin_2); no longer C11.1, D5.1 (K), D7.1 (K), U2.9 (HV)
- net GND: now also J16.2 (Pin_2); no longer U2.10 (GND)
- net GNDREF: now also J10.2 (Pin_2), J13.2 (Pin_2); no longer L2.1, U1.14 (V_IN)
- net I_IN1: now also J15.1 (Pin_1); no longer C8.2, R13.1, R9.2, TP4.1
- net I_IP1: now also J14.1 (Pin_1); no longer C8.1, R10.1, TP3.1
- net STPM10_SCL: now also J9.1 (Pin_1); no longer R21.1, U1.18 (SCL)
- net STPM10_SCS: now also J7.1 (Pin_1); no longer U1.3 (SCS)
- net STPM10_SDA: now also J6.2 (Pin_2); no longer R22.1, U1.19 (SDA)
- net STPM10_SYN: now also J12.1 (Pin_1); no longer R20.1, U1.15 (SYN)
- net V_IP: now also J11.1 (Pin_1); no longer R24.1, R6.1, TP1.1
- new net: J12.2 (Pin_2), R20.1, U1.15 (SYN)
- new net: J9.2 (Pin_2), R21.1, U1.18 (SCL)
- new net: J6.1 (Pin_1), R22.1, U1.19 (SDA)
- new net: J7.2 (Pin_2), U1.3 (SCS)
- new net: J11.2 (Pin_2), R24.1, R6.1, TP1.1
- new net: C8.1, J14.2 (Pin_2), R10.1, TP3.1
- new net: C8.2, J15.2 (Pin_2), R13.1, R9.2, TP4.1
- new net: C11.1, D5.1 (K), D7.1 (K), J8.1 (Pin_1)
- new net: J16.1 (Pin_1), U2.10 (GND)
- new net: J17.2 (Pin_2), U2.9 (HV)
- new net: J10.1 (Pin_1), L2.1
- new net V_IN: J13.1 (Pin_1), U1.14 (V_IN)
Other:
- moved on the sheet: C1, C2, H1, H2, H3, H4, H5, H6, J4, J5, L2, R1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
