File: PCBs/Layer2/Display.kicad_pcb (KiCad board)
At the start: 2 copper layers, 90 x 90 mm, 31 parts, among them J1 Conn_01x12_Male, SW1 SW_Push, SW2 SW_Push, SW3 SW_Push, SW4 SW_Push, SW5 SW_Push, SW6 SW_Push, U2 arduinomini

Commit message: add infrared project
Parts:
- R10, R12, R2, R4, R6, R8: value 100 -> 1k
- SW1, SW2, SW3, SW4, SW5, SW6: footprint TerminalBlock:TerminalBlock_bornier-2_P5.08mm -> Button_Switch_THT:SW_PUSH-12mm_Wuerth-430476085716
- moved H2 193.7 mm to (189.1, 59.0)
- moved H4 158.1 mm to (161.1, 29.8)
- moved H3 106.8 mm to (186.5, 74.3)
- moved H1 73.6 mm to (158.6, 46.3)
- moved R4 59.3 mm to (56.0, 101.7), turned to 270 degrees
- moved C2 58.4 mm to (59.0, 101.7), turned to 270 degrees
- moved R3 53.7 mm to (58.9, 87.7)
- moved C5 52.8 mm to (69.6, 101.7), turned to 270 degrees
- moved C6 51.9 mm to (66.8, 101.7), turned to 270 degrees
- moved C4 51.2 mm to (61.9, 101.7), turned to 270 degrees
- moved R1 51.0 mm to (54.2, 87.7), turned to 90 degrees
- moved C3 45.7 mm to (62.1, 87.7), turned to 90 degrees
- moved R8 38.6 mm to (64.9, 80.2), turned to 90 degrees
- moved R5 36.1 mm to (66.7, 87.7), turned to 270 degrees
- moved R6 35.0 mm to (59.2, 80.6), turned to 90 degrees
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Connections:
- C1 pad 2: Net-(C1-Pad2) -> GND
- C2 pad 2: Net-(C2-Pad2) -> GND
- C3 pad 2: Net-(C3-Pad2) -> GND
- C4 pad 2: Net-(C4-Pad2) -> GND
- C5 pad 2: Net-(C5-Pad2) -> GND
- C6 pad 2: Net-(C6-Pad2) -> GND
- R10 pad 1: Net-(C5-Pad2) -> SW5_ESP
- R10 pad 2: GND -> Net-(R10-Pad2)
- R12 pad 1: Net-(C6-Pad2) -> SW6_ESP
- R12 pad 2: GND -> Net-(R12-Pad2)
- R2 pad 1: Net-(C1-Pad2) -> SW1_Arduino_D13
- R2 pad 2: GND -> Net-(R2-Pad2)
- R4 pad 1: Net-(C2-Pad2) -> Net-(C2-Pad1)
- R4 pad 2: GND -> SW2_Arduino_D12
- R6 pad 1: Net-(C3-Pad2) -> SW3_ESP
- R6 pad 2: GND -> Net-(R6-Pad2)
- R8 pad 1: Net-(C4-Pad2) -> SW4_ESP
- R8 pad 2: GND -> Net-(R8-Pad2)
- SW1 pad 2: SW1_Arduino_D13 -> Net-(R2-Pad2)
- SW2 pad 2: Net-(C2-Pad1) -> SW2_Arduino_D12
- SW3 pad 2: SW3_ESP -> Net-(R6-Pad2)
- SW4 pad 2: SW4_ESP -> Net-(R8-Pad2)
- SW5 pad 2: SW5_ESP -> Net-(R10-Pad2)
- SW6 pad 2: SW6_ESP -> Net-(R12-Pad2)
- U2 pad 15: Net-(C2-Pad1) -> SW2_Arduino_D12
Routing:
- net GND: track 340.9 -> 60.7 mm, vias 3 -> 0
- net +3V3: track 192.1 -> 72.0 mm, vias 3 -> 0
- net OLED_SCL: track 66.6 -> 146.9 mm, vias 1 -> 0
- net SW2_Arduino_D12: track 0.00 -> 79.7 mm, vias 0 -> 1
- net SW5_ESP: track 96.5 -> 34.0 mm, vias 4 -> 0
- net SW3_ESP: track 76.2 -> 22.6 mm
- net Net-(R2-Pad2): track 0.00 -> 51.4 mm
- net SW4_ESP: track 82.9 -> 31.9 mm, vias 0 -> 2
- net OLED_SDA: track 83.8 -> 132.4 mm, vias 1 -> 0
- net Net-(R6-Pad2): track 0.00 -> 44.9 mm
- net SW6_ESP: track 44.0 -> 0.00 mm
- net Net-(C2-Pad1): track 52.3 -> 14.0 mm
- net Net-(C3-Pad2): track 35.3 -> 0.00 mm
- net Net-(C1-Pad2): track 29.4 -> 0.00 mm
- net Net-(R8-Pad2): track 0.00 -> 28.8 mm
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- removed copper zone on B.Cu, net GND
- removed copper zone on F.Cu, net GND
Other:
- board size 90 x 90 mm -> 90 x 110 mm

Commit message: display update
Parts:
- removed DS1: 128x64_OLED_Display-Arduino_Module_Custom, Connector_PinHeader_2.54mm:PinHeader_1x04_P2.54mm_Vertical
- removed U2: arduinomini, Arduino_mini:Arduinomini
- added J2: Conn_01x08_Male, Connector_PinHeader_2.54mm:PinHeader_1x08_P2.54mm_Vertical, F.Cu at (39.8, 12.2)
- added U1: arduinopromini, arduinopromini:arduinopromini, F.Cu at (7.45, 24.7)
- moved SW2 48.5 mm to (68.9, 35.0)
- moved SW3 48.5 mm to (83.3, 34.8)
- moved SW1 48.5 mm to (54.6, 35.0)
- moved C3 34.4 mm to (27.8, 90.0)
- moved C5 34.4 mm to (35.3, 104.0)
- moved C6 34.4 mm to (32.5, 103.9)
- moved R10 34.4 mm to (31.1, 75.9)
- moved R11 34.4 mm to (41.2, 88.9)
- moved R6 34.4 mm to (24.9, 82.9)
- moved R8 34.4 mm to (30.6, 82.5)
- moved C1 34.4 mm to (20.7, 82.9)
- moved C2 34.4 mm to (24.7, 104.0)
- moved C4 34.4 mm to (27.6, 104.0)
- moved R1 34.4 mm to (19.9, 90.0)
- moved R2 34.4 mm to (16.6, 82.9)
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Routing:
- net OLED_SCL: track 146.9 -> 0.00 mm
- net OLED_SDA: track 132.4 -> 0.00 mm
- net SW2_Arduino_D12: track 79.7 -> 0.00 mm, vias 1 -> 0
- net +3V3: track 72.0 -> 0.00 mm
- net SW1_Arduino_D13: track 64.3 -> 0.00 mm
- net GND: track 60.7 -> 0.00 mm
- net ESP32_TX: track 52.2 -> 0.00 mm, vias 1 -> 0
- net Net-(R2-Pad2): track 51.4 -> 0.00 mm
- net ESP32_RX: track 50.8 -> 0.00 mm, vias 1 -> 0
- net +5V: track 46.0 -> 0.00 mm
- net Net-(R6-Pad2): track 44.9 -> 0.00 mm
- net SW5_ESP: track 34.0 -> 0.00 mm
- net SW4_ESP: track 31.9 -> 0.00 mm, vias 2 -> 0
- net Net-(R8-Pad2): track 28.8 -> 0.00 mm
- net SW3_ESP: track 22.6 -> 0.00 mm
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
Commit message: layer 2 update
Parts:
- U1: moved to B.Cu
- moved H2 194.0 mm to (3.00, 4.00)
- moved H1 167.4 mm to (3.00, 108.0)
- moved H3 105.1 mm to (87.0, 108.0)
- moved H4 78.5 mm to (87.0, 4.00)
- moved SW1 57.8 mm to (62.3, 92.3)
- moved SW5 53.1 mm to (29.2, 92.2)
- moved SW4 52.9 mm to (15.0, 92.2)
- moved SW6 51.6 mm to (45.9, 92.3)
- moved C2 31.2 mm to (13.3, 74.9)
- moved SW2 28.7 mm to (40.3, 38.0)
- moved R5 28.6 mm to (58.0, 77.4)
- moved R6 28.6 mm to (50.5, 70.3)
- moved C1 28.6 mm to (46.4, 70.3)
- moved C3 28.6 mm to (53.5, 77.4)
- moved R2 28.6 mm to (42.3, 70.3)
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Routing:
- net GND: track 0.00 -> 326.8 mm, vias 0 -> 2
- net +3V3: track 0.00 -> 188.8 mm, vias 0 -> 4
- net SW4_ESP: track 0.00 -> 111.3 mm, vias 0 -> 3
- net SW5_ESP: track 0.00 -> 99.5 mm, vias 0 -> 1
- net SW6_ESP: track 0.00 -> 91.3 mm
- net ESP32_RX: track 0.00 -> 86.1 mm
- net ESP32_TX: track 0.00 -> 85.9 mm
- net +5V: track 0.00 -> 85.4 mm
- net SW2_Arduino_D12: track 0.00 -> 72.5 mm
- net SW1_Arduino_D13: track 0.00 -> 66.3 mm, vias 0 -> 2
- net SDA: track 0.00 -> 54.7 mm
- net SW3_ESP: track 0.00 -> 51.9 mm, vias 0 -> 2
- net Net-(C2-Pad1): track 0.00 -> 51.0 mm, vias 0 -> 2
- net Net-(R12-Pad2): track 0.00 -> 46.1 mm
- net Net-(R2-Pad2): track 0.00 -> 39.8 mm, vias 0 -> 1
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- added copper zone on B.Cu, net GND
- added copper zone on F.Cu, net GND

Commit message: WIP
Parts:
- added H5: MountingHole, MountingHole:MountingHole_2.7mm_M2.5_DIN965, F.Cu at (104.0, 71.0)
- added H6: MountingHole, MountingHole:MountingHole_2.7mm_M2.5_DIN965, F.Cu at (20.0, 70.0)
- moved R6 26.2 mm to (67.5, 90.3)
- moved C6 26.2 mm to (44.8, 99.8)
- moved U1 26.2 mm to (41.1, 67.7)
- moved C1 26.2 mm to (63.4, 90.3)
- moved C2 26.2 mm to (30.3, 94.9)
- moved C3 26.2 mm to (70.5, 97.4)
- moved C4 26.2 mm to (33.1, 101.9)
- moved C5 26.2 mm to (47.6, 99.8)
- moved H1 26.2 mm to (20.0, 128.0)
- moved H3 26.2 mm to (104.0, 128.0)
- moved J1 26.2 mm to (103.3, 123.0)
- moved J2 26.2 mm to (56.8, 32.2)
- moved R1 26.2 mm to (62.5, 97.4)
- moved R10 26.2 mm to (46.2, 106.6)
- moved R11 26.2 mm to (83.9, 96.3)
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Other:
- board size 90 x 110 mm -> 90 x 113 mm
